Commit message: Use updated cybertech macro

File: src/cybertech_mock/description/kuka_cybertech.urdf.xacro (robot description, xacro)
@@ -19,4 +19,5 @@
   <xacro:arg name="pitch" default="0" />
   <xacro:arg name="yaw" default="0" />
+  <link name="world" />
   <xacro:kuka_cybertech_ros2_control name="$(arg prefix)kr16_r2010_2"
     driver_version="$(arg driver_version)" client_ip="$(arg client_ip)"
@@ -24,5 +25,6 @@
     mode="$(arg mode)" use_gpio="$(arg use_gpio)" roundtrip_time="$(arg roundtrip_time)"
     verify_robot_model="$(arg verify_robot_model)" />
-  <xacro:kuka_kr16_r2010_2_robot prefix="$(arg prefix)" package_name="kuka_cybertech_support">
+  <xacro:kuka_kr16_r2010_2_robot prefix="$(arg prefix)" package_name="kuka_cybertech_support"
+    parent="world">
     <origin xyz="$(arg x) $(arg y) $(arg z)" rpy="$(arg roll) $(arg pitch) $(arg yaw)" />
   </xacro:kuka_kr16_r2010_2_robot>
